File: usb-rj45-serial-dongle.sch (EAGLE design)
At the start: 16 parts, among them IC1 MAX202ECWE, J1 RJHSE-5381, J2 USBPCB_NOPASTE, U1 CP2102N-A01-GQFN20R, U2 SP0503BAHTG

Commit message: Board updates, silkscreen cleanup and component changes
Board updates:
- GND plane stitching changed to a more general pattern rather than closely stitched to signal lines, since we aren't doing RF
- GND plane optimizations (bottom layer no longer separated into 2 distinct planes)
- Reduced size of board

Silkscreen cleanup:
- Removed values
- Rotated names and changed size/font to fit better and avoid vias (Seeed Fusion doesn't do blind via silkscreen well)

Component Changes:
- J1: RJHSE-5381 (shielded RJ45) replaced with RJHSE-5081 (unshielded RJ45) for smaller footprint and lower cost
- R3: Changed from Seeed OPL 0402 1KΩ 1% to 5% tolerance part due to value error (0R) on the 1% part
Parts:
- J1: value RJHSE-5381 -> RJHSE-5081; device RJHSE-5381:RJHSE-5381 -> RJHSE-5081:RJHSE-5081
- R3: value 0R -> 1K; device OPL_Resistor:SMD-RES-1K-1%-1/16W(0402) -> OPL_Resistor:SMD-RES-1K-5%-1/16W(0402)
Connections:
- net GND: no longer J1.S1, J1.S2
Changed lines of the file:
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@@
 <parts>
 <part name="U1" library="CP2102N-A01-GQFN20R" deviceset="CP2102N-A01-GQFN20R" device=""/>
-<part name="J1" library="RJHSE-5381" deviceset="RJHSE-5381" device=""/>
+<part name="J1" library="RJHSE-5081" deviceset="RJHSE-5081" device=""/>
 <part name="GND1" library="supply1" library_urn="urn:adsk.eagle:library:371" deviceset="GND" device=""/>
 <part name="C1" library="OPL_Capacitor" library_urn="urn:adsk.eagle:library:8004261" deviceset="CERAMIC-4.7UF-6.3V-20%-X5R(0402)" device="" package3d_urn="urn:adsk.eagle:package:8004285/1" value="4.7uf"/>
 <part name="C2" library="OPL_Capacitor" library_urn="urn:adsk.eagle:library:8004261" deviceset="CERAMIC-100NF-25V-10%-X7R(0402)" device="" package3d_urn="urn:adsk.eagle:package:8004285/1" value="100nf"/>
 <part name="GND3" library="supply1" library_urn="urn:adsk.eagle:library:371" deviceset="GND" device=""/>
-<part name="R3" library="OPL_Resistor" library_urn="urn:adsk.eagle:library:8004883" deviceset="SMD-RES-1K-1%-1/16W(0402)" device="" package3d_urn="urn:adsk.eagle:package:8004940/1" value="0R"/>
+<part name="R3" library="OPL_Resistor" library_urn="urn:adsk.eagle:library:8004883" deviceset="SMD-RES-1K-5%-1/16W(0402)" device="" package3d_urn="urn:adsk.eagle:package:8004940/1" value="1K"/>
 <part name="C3" library="OPL_Capacitor" library_urn="urn:adsk.eagle:library:8004261" deviceset="CERAMIC-4.7UF-6.3V-20%-X5R(0402)" device="" package3d_urn="urn:adsk.eagle:package:8004285/1" value="4.7uf"/>
 <part name="C4" library="OPL_Capacitor" library_urn="urn:adsk.eagle:library:8004261" deviceset="CERAMIC-100NF-25V-10%-X7R(0402)" device="" package3d_urn="urn:adsk.eagle:package:8004285/1" value="100nf"/>
@@
 <part name="R6" library="OPL_Resistor" library_urn="urn:adsk.eagle:library:8004883" deviceset="SMD-RES-330R-1%-1/16W(0402)" device="" package3d_urn="urn:adsk.eagle:package:8004940/1" value="330R"/>
 <part name="R7" library="OPL_Resistor" library_urn="urn:adsk.eagle:library:8004883" deviceset="SMD-RES-330R-1%-1/16W(0402)" device="" package3d_urn="urn:adsk.eagle:package:8004940/1" value="330R"/>
-<part name="GND6" library="supply1" library_urn="urn:adsk.eagle:library:371" deviceset="GND" device=""/>
 <part name="J2" library="SparkFun-Connectors" deviceset="USB" device="PCB_NOPASTE"/>
 <part name="GND7" library="supply1" library_urn="urn:adsk.eagle:library:371" deviceset="GND" device=""/>
@@
 <attribute name="NAME" x="24.13" y="67.31" size="1.27" layer="95" ratio="10"/>
 <attribute name="VALUE" x="24.13" y="63.5" size="1.27" layer="96" ratio="10"/>
-</instance>
-<instance part="GND6" gate="1" x="33.02" y="55.88" smashed="yes">
-<attribute name="VALUE" x="30.48" y="53.34" size="1.778" layer="96"/>
 </instance>
 <instance part="J2" gate="G$1" x="88.9" y="119.38" smashed="yes">
@@
 </segment>
 <segment>
-<pinref part="J1" gate="G$1" pin="S1"/>
-<wire x1="35.56" y1="74.93" x2="33.02" y2="74.93" width="0.1524" layer="91"/>
-<wire x1="33.02" y1="74.93" x2="33.02" y2="72.39" width="0.1524" layer="91"/>
-<pinref part="J1" gate="G$1" pin="S2"/>
-<wire x1="33.02" y1="72.39" x2="35.56" y2="72.39" width="0.1524" layer="91"/>
-<wire x1="33.02" y1="72.39" x2="33.02" y2="58.42" width="0.1524" layer="91"/>
-<pinref part="GND6" gate="1" pin="GND"/>
-</segment>
-<segment>

Commit message: Renumber resistors to start from R1
Parts:
- removed R7: 330R, OPL_Resistor:SMD-RES-330R-1%-1/16W(0402)
- added R1: 1K, OPL_Resistor:SMD-RES-1K-5%-1/16W(0402)
- R3: value 1K -> 330R; device OPL_Resistor:SMD-RES-1K-5%-1/16W(0402) -> OPL_Resistor:SMD-RES-330R-1%-1/16W(0402)
- renumbered R6 to R2
Connections:
- net 3V3: now also R1.1; no longer R7.1
- net N$2: now also R1.2; no longer R3.2
- net N$3: now also R3.2; no longer R7.2
Other:
- moved on the sheet: R3
Changed lines of the file:
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@@
 <part name="C2" library="OPL_Capacitor" library_urn="urn:adsk.eagle:library:8004261" deviceset="CERAMIC-100NF-25V-10%-X7R(0402)" device="" package3d_urn="urn:adsk.eagle:package:8004285/1" value="100nf"/>
 <part name="GND3" library="supply1" library_urn="urn:adsk.eagle:library:371" deviceset="GND" device=""/>
-<part name="R3" library="OPL_Resistor" library_urn="urn:adsk.eagle:library:8004883" deviceset="SMD-RES-1K-5%-1/16W(0402)" device="" package3d_urn="urn:adsk.eagle:package:8004940/1" value="1K"/>
+<part name="R1" library="OPL_Resistor" library_urn="urn:adsk.eagle:library:8004883" deviceset="SMD-RES-1K-5%-1/16W(0402)" device="" package3d_urn="urn:adsk.eagle:package:8004940/1" value="1K"/>
 <part name="C3" library="OPL_Capacitor" library_urn="urn:adsk.eagle:library:8004261" deviceset="CERAMIC-4.7UF-6.3V-20%-X5R(0402)" device="" package3d_urn="urn:adsk.eagle:package:8004285/1" value="4.7uf"/>
 <part name="C4" library="OPL_Capacitor" library_urn="urn:adsk.eagle:library:8004261" deviceset="CERAMIC-100NF-25V-10%-X7R(0402)" device="" package3d_urn="urn:adsk.eagle:package:8004285/1" value="100nf"/>
 <part name="GND4" library="supply1" library_urn="urn:adsk.eagle:library:371" deviceset="GND" device=""/>
-<part name="R6" library="OPL_Resistor" library_urn="urn:adsk.eagle:library:8004883" deviceset="SMD-RES-330R-1%-1/16W(0402)" device="" package3d_urn="urn:adsk.eagle:package:8004940/1" value="330R"/>
-<part name="R7" library="OPL_Resistor" library_urn="urn:adsk.eagle:library:8004883" deviceset="SMD-RES-330R-1%-1/16W(0402)" device="" package3d_urn="urn:adsk.eagle:package:8004940/1" value="330R"/>
+<part name="R2" library="OPL_Resistor" library_urn="urn:adsk.eagle:library:8004883" deviceset="SMD-RES-330R-1%-1/16W(0402)" device="" package3d_urn="urn:adsk.eagle:package:8004940/1" value="330R"/>
+<part name="R3" library="OPL_Resistor" library_urn="urn:adsk.eagle:library:8004883" deviceset="SMD-RES-330R-1%-1/16W(0402)" device="" package3d_urn="urn:adsk.eagle:package:8004940/1" value="330R"/>
 <part name="J2" library="SparkFun-Connectors" deviceset="USB" device="PCB_NOPASTE"/>
 <part name="GND7" library="supply1" library_urn="urn:adsk.eagle:library:371" deviceset="GND" device=""/>
@@
 <attribute name="VALUE" x="96.52" y="2.54" size="1.778" layer="96"/>
 </instance>
-<instance part="R3" gate="G$1" x="15.24" y="20.32" smashed="yes">
+<instance part="R1" gate="G$1" x="15.24" y="20.32" smashed="yes">
 <attribute name="NAME" x="11.43" y="21.59" size="1.27" layer="95" ratio="10"/>
 <attribute name="VALUE" x="11.43" y="17.78" size="1.27" layer="96" ratio="10"/>
@@
 <attribute name="VALUE" x="83.82" y="2.54" size="1.778" layer="96"/>
 </instance>
-<instance part="R6" gate="G$1" x="27.94" y="81.28" smashed="yes">
+<instance part="R2" gate="G$1" x="27.94" y="81.28" smashed="yes">
 <attribute name="NAME" x="24.13" y="82.55" size="1.27" layer="95" ratio="10"/>
 <attribute name="VALUE" x="24.13" y="78.74" size="1.27" layer="96" ratio="10"/>
 </instance>
-<instance part="R7" gate="G$1" x="27.94" y="66.04" smashed="yes">
+<instance part="R3" gate="G$1" x="27.94" y="66.04" smashed="yes">
 <attribute name="NAME" x="24.13" y="67.31" size="1.27" layer="95" ratio="10"/>
 <attribute name="VALUE" x="24.13" y="63.5" size="1.27" layer="96" ratio="10"/>
@@
 </segment>
 <segment>
-<pinref part="R3" gate="G$1" pin="1"/>
+<pinref part="R1" gate="G$1" pin="1"/>
 <wire x1="11.43" y1="20.32" x2="10.16" y2="20.32" width="0.1524" layer="91"/>
 <label x="10.16" y="20.32" size="1.778" layer="95" rot="R180" xref="yes"/>
 </segment>
 <segment>
-<pinref part="R7" gate="G$1" pin="1"/>
+<pinref part="R3" gate="G$1" pin="1"/>
 <wire x1="24.13" y1="66.04" x2="22.86" y2="66.04" width="0.1524" layer="91"/>
 <wire x1="22.86" y1="66.04" x2="22.86" y2="81.28" width="0.1524" layer="91"/>
-<pinref part="R6" gate="G$1" pin="1"/>
+<pinref part="R2" gate="G$1" pin="1"/>
 <wire x1="22.86" y1="81.28" x2="24.13" y2="81.28" width="0.1524" layer="91"/>
 <wire x1="22.86" y1="81.28" x2="22.86" y2="86.36" width="0.1524" layer="91"/>
@@
 <segment>
 <pinref part="U1" gate="G$1" pin="RST"/>
-<pinref part="R3" gate="G$1" pin="2"/>
+<pinref part="R1" gate="G$1" pin="2"/>
 <wire x1="20.32" y1="20.32" x2="19.05" y2="20.32" width="0.1524" layer="91"/>
 </segment>
@@
 <net name="N$3" class="0">
 <segment>
-<pinref part="R7" gate="G$1" pin="2"/>
+<pinref part="R3" gate="G$1" pin="2"/>
 <pinref part="J1" gate="G$1" pin="12"/>
 <wire x1="31.75" y1="66.04" x2="31.75" y2="64.77" width="0.1524" layer="91"/>
@@
 <net name="N$5" class="0">
 <segment>
-<pinref part="R6" gate="G$1" pin="2"/>
+<pinref part="R2" gate="G$1" pin="2"/>
 <pinref part="J1" gate="G$1" pin="10"/>
 <wire x1="31.75" y1="81.28" x2="31.75" y2="80.01" width="0.1524" layer="91"/>

Commit message: Renumber IC1 and other ICs to be in sequence with prefix "U"
Parts:
- removed IC1: MAX202ECWE, maxim:MAX202ECWE
- added U3: SP0503BAHTG, littlefuse:SP0503BAHTG
- U2: value SP0503BAHTG -> MAX202ECWE; device littlefuse:SP0503BAHTG -> maxim:MAX202ECWE
Connections:
- net CTS: now also U2G$1.R2IN; no longer IC1G$1.R2IN
- net GND: now also U3.GND; no longer U2.GND
- net N$1: now also U2G$1.C1+; no longer IC1G$1.C1+
- net N$4: now also U2G$1.C2+; no longer IC1G$1.C2+
- net N$6: now also U2G$1.C1-; no longer IC1G$1.C1-
- net N$7: now also U2G$1.C2-; no longer IC1G$1.C2-
- net N$8: now also U2G$1.V+; no longer IC1G$1.V+
- net N$9: now also U2G$1.V-; no longer IC1G$1.V-
- net RTS: now also U2G$1.T2OUT; no longer IC1G$1.T2OUT
- net RXD: now also U2G$1.R1IN; no longer IC1G$1.R1IN
- net TXD: now also U2G$1.T1OUT; no longer IC1G$1.T1OUT
- net UART_CTS: now also U2G$1.R1OUT; no longer IC1G$1.R1OUT
- net UART_RTS: now also U2G$1.T2IN; no longer IC1G$1.T2IN
- net UART_RXD: now also U2G$1.R2OUT; no longer IC1G$1.R2OUT
- net UART_TXD: now also U2G$1.T1IN; no longer IC1G$1.T1IN
- net USBDN: now also U3.B; no longer U2.B
- net USBDP: now also U3.C; no longer U2.C
- net VCC: now also U3.A; no longer U2.A
Changed lines of the file:
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@@
 <part name="J2" library="SparkFun-Connectors" deviceset="USB" device="PCB_NOPASTE"/>
 <part name="GND7" library="supply1" library_urn="urn:adsk.eagle:library:371" deviceset="GND" device=""/>
-<part name="IC1" library="maxim" library_urn="urn:adsk.eagle:library:269" deviceset="MAX202ECWE" device="" package3d_urn="urn:adsk.eagle:package:17518/2"/>
+<part name="U2" library="maxim" library_urn="urn:adsk.eagle:library:269" deviceset="MAX202ECWE" device="" package3d_urn="urn:adsk.eagle:package:17518/2"/>
 <part name="C5" library="OPL_Capacitor" library_urn="urn:adsk.eagle:library:8004261" deviceset="CERAMIC-100NF-25V-10%-X7R(0402)" device="" package3d_urn="urn:adsk.eagle:package:8004285/1" value="100nf"/>
 <part name="C6" library="OPL_Capacitor" library_urn="urn:adsk.eagle:library:8004261" deviceset="CERAMIC-100NF-25V-10%-X7R(0402)" device="" package3d_urn="urn:adsk.eagle:package:8004285/1" value="100nf"/>
@@
 <part name="C8" library="OPL_Capacitor" library_urn="urn:adsk.eagle:library:8004261" deviceset="CERAMIC-100NF-25V-10%-X7R(0402)" device="" package3d_urn="urn:adsk.eagle:package:8004285/1" value="100nf"/>
 <part name="GND2" library="supply1" library_urn="urn:adsk.eagle:library:371" deviceset="GND" device=""/>
-<part name="U2" library="littlefuse" deviceset="SP0503BAHTG" device=""/>
+<part name="U3" library="littlefuse" deviceset="SP0503BAHTG" device=""/>
 <part name="GND5" library="supply1" library_urn="urn:adsk.eagle:library:371" deviceset="GND" device=""/>
 </parts>
@@
 <attribute name="VALUE" x="78.74" y="111.76" size="1.778" layer="96"/>
 </instance>
-<instance part="IC1" gate="G$1" x="124.46" y="63.5" smashed="yes">
+<instance part="U2" gate="G$1" x="124.46" y="63.5" smashed="yes">
 <attribute name="NAME" x="114.3" y="79.375" size="1.778" layer="95"/>
 <attribute name="VALUE" x="114.3" y="43.18" size="1.778" layer="96"/>
@@
 <attribute name="VALUE" x="147.32" y="60.96" size="1.778" layer="96"/>
 </instance>
-<instance part="U2" gate="G$1" x="127" y="96.52" smashed="yes" rot="R270">
+<instance part="U3" gate="G$1" x="127" y="96.52" smashed="yes" rot="R270">
 <attribute name="NAME" x="124.44" y="91.944" size="1.016" layer="95"/>
 <attribute name="VALUE" x="124.44" y="89.92" size="1.016" layer="96"/>
@@
 </segment>
 <segment>
-<pinref part="U2" gate="G$1" pin="GND"/>
+<pinref part="U3" gate="G$1" pin="GND"/>
 <wire x1="124.46" y1="101.6" x2="124.46" y2="104.14" width="0.1524" layer="91"/>
 <pinref part="GND5" gate="1" pin="GND"/>
@@
 </segment>
 <segment>
-<pinref part="IC1" gate="G$1" pin="R1IN"/>
+<pinref part="U2" gate="G$1" pin="R1IN"/>
 <wire x1="139.7" y1="50.8" x2="142.24" y2="50.8" width="0.1524" layer="91"/>
 <label x="142.24" y="50.8" size="1.778" layer="95" xref="yes"/>
@@
 </segment>
 <segment>
-<pinref part="IC1" gate="G$1" pin="R2IN"/>
+<pinref part="U2" gate="G$1" pin="R2IN"/>
 <wire x1="139.7" y1="48.26" x2="142.24" y2="48.26" width="0.1524" layer="91"/>
 <label x="142.24" y="48.26" size="1.778" layer="95" xref="yes"/>
@@
 </segment>
 <segment>
-<pinref part="IC1" gate="G$1" pin="T1OUT"/>
+<pinref part="U2" gate="G$1" pin="T1OUT"/>
 <wire x1="139.7" y1="55.88" x2="142.24" y2="55.88" width="0.1524" layer="91"/>
 <label x="142.24" y="55.88" size="1.778" layer="95" xref="yes"/>
@@
 </segment>
 <segment>
-<pinref part="IC1" gate="G$1" pin="T2OUT"/>
+<pinref part="U2" gate="G$1" pin="T2OUT"/>
 <wire x1="139.7" y1="53.34" x2="142.24" y2="53.34" width="0.1524" layer="91"/>
 <label x="142.24" y="53.34" size="1.778" layer="95" xref="yes"/>
@@
 </segment>
 <segment>
-<pinref part="IC1" gate="G$1" pin="T1IN"/>
+<pinref part="U2" gate="G$1" pin="T1IN"/>
 <wire x1="109.22" y1="55.88" x2="106.68" y2="55.88" width="0.1524" layer="91"/>
 <label x="106.68" y="55.88" size="1.778" layer="95" rot="R180" xref="yes"/>
@@
 </segment>
 <segment>
-<pinref part="IC1" gate="G$1" pin="R2OUT"/>
+<pinref part="U2" gate="G$1" pin="R2OUT"/>
 <wire x1="109.22" y1="48.26" x2="106.68" y2="48.26" width="0.1524" layer="91"/>
 <label x="106.68" y="48.26" size="1.778" layer="95" rot="R180" xref="yes"/>
@@
 </segment>
 <segment>
-<pinref part="U2" gate="G$1" pin="A"/>
+<pinref part="U3" gate="G$1" pin="A"/>
 <wire x1="127" y1="99.06" x2="134.62" y2="99.06" width="0.1524" layer="91"/>
 <label x="134.62" y="99.06" size="1.778" layer="95" xref="yes"/>
@@
 </segment>
 <segment>
-<pinref part="IC1" gate="G$1" pin="T2IN"/>
+<pinref part="U2" gate="G$1" pin="T2IN"/>
 <wire x1="109.22" y1="53.34" x2="106.68" y2="53.34" width="0.1524" layer="91"/>
 <label x="106.68" y="53.34" size="1.778" layer="95" rot="R180" xref="yes"/>
@@
 </segment>
 <segment>
-<pinref part="IC1" gate="G$1" pin="R1OUT"/>
+<pinref part="U2" gate="G$1" pin="R1OUT"/>
 <wire x1="109.22" y1="50.8" x2="106.68" y2="50.8" width="0.1524" layer="91"/>
 <label x="106.68" y="50.8" size="1.778" layer="95" rot="R180" xref="yes"/>
@@
 </segment>
 <segment>
-<pinref part="U2" gate="G$1" pin="C"/>
+<pinref part="U3" gate="G$1" pin="C"/>
 <wire x1="132.08" y1="93.98" x2="134.62" y2="93.98" width="0.1524" layer="91"/>
 <label x="134.62" y="93.98" size="1.778" layer="95" xref="yes"/>
@@
 </segment>
 <segment>
-<pinref part="U2" gate="G$1" pin="B"/>
+<pinref part="U3" gate="G$1" pin="B"/>
 <wire x1="129.54" y1="96.52" x2="134.62" y2="96.52" width="0.1524" layer="91"/>
 <label x="134.62" y="96.52" size="1.778" layer="95" xref="yes"/>
@@
 <net name="N$1" class="0">
 <segment>
-<pinref part="IC1" gate="G$1" pin="C1+"/>
+<pinref part="U2" gate="G$1" pin="C1+"/>
 <pinref part="C5" gate="G$1" pin="2"/>
 <wire x1="109.22" y1="76.2" x2="107.95" y2="76.2" width="0.1524" layer="91"/>
@@
 <net name="N$4" class="0">
 <segment>
-<pinref part="IC1" gate="G$1" pin="C2+"/>
+<pinref part="U2" gate="G$1" pin="C2+"/>
 <pinref part="C6" gate="G$1" pin="2"/>
 <wire x1="109.22" y1="66.04" x2="107.95" y2="66.04" width="0.1524" layer="91"/>
@@
 <wire x1="100.33" y1="76.2" x2="99.06" y2="76.2" width="0.1524" layer="91"/>
 <wire x1="99.06" y1="76.2" x2="99.06" y2="71.12" width="0.1524" layer="91"/>
-<pinref part="IC1" gate="G$1" pin="C1-"/>
+<pinref part="U2" gate="G$1" pin="C1-"/>
 <wire x1="99.06" y1="71.12" x2="109.22" y2="71.12" width="0.1524" layer="91"/>
 </segment>
@@
 <wire x1="100.33" y1="66.04" x2="99.06" y2="66.04" width="0.1524" layer="91"/>
 <wire x1="99.06" y1="66.04" x2="99.06" y2="60.96" width="0.1524" layer="91"/>
-<pinref part="IC1" gate="G$1" pin="C2-"/>
+<pinref part="U2" gate="G$1" pin="C2-"/>
 <wire x1="99.06" y1="60.96" x2="109.22" y2="60.96" width="0.1524" layer="91"/>
 </segment>
@@
 <net name="N$8" class="0">
 <segment>
-<pinref part="IC1" gate="G$1" pin="V+"/>
+<pinref part="U2" gate="G$1" pin="V+"/>
 <pinref part="C7" gate="G$1" pin="1"/>
 <wire x1="139.7" y1="73.66" x2="140.97" y2="73.66" width="0.1524" layer="91"/>
@@
 <net name="N$9" class="0">
 <segment>
-<pinref part="IC1" gate="G$1" pin="V-"/>
+<pinref part="U2" gate="G$1" pin="V-"/>
 <pinref part="C8" gate="G$1" pin="1"/>
 <wire x1="139.7" y1="68.58" x2="140.97" y2="68.58" width="0.1524" layer="91"/>

Commit message: Use CP2102 TXT/RXT pins to drive LEDs, thanks @MatsK for pointing this feature out
Connections:
- new net RXT_LED: J1.9, U1.GPIO.3/RXT
- new net TXT_LED: J1.11, U1.GPIO.2/TXT
- net UART_RXD: no longer J1.9
- net UART_TXD: no longer J1.11
Changed lines of the file:
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@@
-</segment>
-<segment>
-<pinref part="J1" gate="G$1" pin="11"/>
-<wire x1="35.56" y1="67.31" x2="27.94" y2="67.31" width="0.1524" layer="91"/>
-<wire x1="27.94" y1="67.31" x2="27.94" y2="86.36" width="0.1524" layer="91"/>
-<label x="27.94" y="86.36" size="1.778" layer="95" rot="R90" xref="yes"/>
 </segment>
 <segment>
@@
 <wire x1="20.32" y1="40.64" x2="17.78" y2="40.64" width="0.1524" layer="91"/>
 <label x="17.78" y="40.64" size="1.778" layer="95" rot="R180" xref="yes"/>
-</segment>
-<segment>
-<pinref part="J1" gate="G$1" pin="9"/>
-<wire x1="35.56" y1="82.55" x2="33.02" y2="82.55" width="0.1524" layer="91"/>
-<wire x1="33.02" y1="82.55" x2="33.02" y2="86.36" width="0.1524" layer="91"/>
-<label x="33.02" y="86.36" size="1.778" layer="95" rot="R90" xref="yes"/>
 </segment>
 <segment>
@@
 </segment>
 </net>
+<net name="RXT_LED" class="0">
+<segment>
+<pinref part="U1" gate="G$1" pin="GPIO.3/RXT"/>
+<wire x1="55.88" y1="22.86" x2="58.42" y2="22.86" width="0.1524" layer="91"/>
+<label x="58.42" y="22.86" size="1.778" layer="95" xref="yes"/>
+</segment>
+<segment>
+<pinref part="J1" gate="G$1" pin="9"/>
+<wire x1="35.56" y1="82.55" x2="33.02" y2="82.55" width="0.1524" layer="91"/>
+<wire x1="33.02" y1="82.55" x2="33.02" y2="86.36" width="0.1524" layer="91"/>
+<label x="33.02" y="86.36" size="1.778" layer="95" rot="R90" xref="yes"/>
+</segment>
+</net>
+<net name="TXT_LED" class="0">
+<segment>
+<pinref part="U1" gate="G$1" pin="GPIO.2/TXT"/>
+<wire x1="55.88" y1="20.32" x2="58.42" y2="20.32" width="0.1524" layer="91"/>
+<label x="58.42" y="20.32" size="1.778" layer="95" xref="yes"/>
+</segment>
+<segment>
+<pinref part="J1" gate="G$1" pin="11"/>
+<wire x1="35.56" y1="67.31" x2="27.94" y2="67.31" width="0.1524" layer="91"/>
+<wire x1="27.94" y1="67.31" x2="27.94" y2="86.36" width="0.1524" layer="91"/>
+<label x="27.94" y="86.36" size="1.778" layer="95" rot="R90" xref="yes"/>
+</segment>
+</net>
